File: silkscreen_pcb.kicad_pcb (KiCad board)
At the start: 2 copper layers, 60 x 111.3 mm, 183 parts, among them J1 USB_C_Receptacle, J2 FH34SRJ-24S-0.5SH_50_, J3 FH34SRJ-6S-0.5SH_50_, J4 FH34SRJ-6S-0.5SH_50_, J5 Conn_01x02, J6 PPPC062LJBN-RC, J7 Micro_SD_Card, Q1 FS8205A, Q2 AO3401A, Q3 AO3401A, Q4 IRLML6346TRPBF, Q5 BSS138, Q6 BSS138, Q7 AO3401A, Q8 AO3401A, Q9 BSS138, SW1 SW_Push, SW10 SW_Push, SW11 SW_Push, SW2 SW_Push, SW3 SW_Push, SW4 SW_Push, SW5 SW_Push, SW6 SW_Push, SW7 SW_Push, SW8 SW_Push, SW9 SW_Push, U1 TPD4E1U06DBVR, U10 TPS923610DRLR, U11 TP4056-42-ESOP8, U12 74LVC1G04, U13 DS3231MZ, U2 TPS2116DRL, U3 TLV75533PDBV, U4 ESP32-S3-WROOM-1, U5 DW01A, U6 TPD4E1U06DBVR, U7 TPD4E1U06DBVR, U8 TPD4E1U06DBVR, U9 TPD4E1U06DBVR

Commit message: Other-fab ordering files, optional front-mounted bottom buttons, W-/C- reroute
- fabrication/make_fab_files.py and production/other_fabs/: PCBWay and NextPCB
  BOMs (MPN-keyed), raw KiCad bottom-side placement file, NextPCB centroid CSV (NextPCB sample layout) and a
  legible bottom-side assembly drawing; README section "Ordering from PCBWay or
  NextPCB" and JLC step 4/6 corrections
- Optional front-mounted bottom buttons: open solder-bridge tabs beside the mounting
  holes of SW2/SW3/SW8/SW9 (GND and ladder node), with solder-mask windows on the
  tab tips, so a hand-fitted APEM MJTP1243 can replace the right-angle switch.
  Documented in docs/HARDWARE.md 9.1.1; never bridged with an MJTP1117/TS365ZJ fitted
- W- and C- frontlight returns rerouted out of the bottom button strip
- Gerbers and netlist regenerated with the Fabrication Toolkit for this board state;
  other-fab files re-run against it; DRC exclusions for the intentionally open tab tips

- NextPCB centroid lists every fitted BOM part, through-hole included, so its designators
  match nextpcb_bom.csv (NextPCB rejects a PnP/BOM designator mismatch)
- JLC v4 upload BOM: merge the two pairs of lines that shared a JLC part number
  (C14663: C7/C24/C30/C31/C33/C36; C28323: C18/C19/C20) so JLC matches all of them
Routing:
- net C-: track 219.3 -> 187.9 mm, vias 4 -> 3
- net W-: track 191.9 -> 172.9 mm, vias 3 -> 2
- net LED_SW: track 198.5 -> 180.4 mm
- net GND: track 30.8 -> 48.8 mm
- net Net-(R18-Pad1): track 32.5 -> 37.2 mm
- net Net-(R19-Pad1): track 22.3 -> 26.6 mm
- net Net-(R60-Pad1): track 59.7 -> 64.0 mm
- net Net-(R20-Pad1): track 13.8 -> 18.1 mm

Commit message: Final-review revision: DW01A filters, J6 fuse, alternate RTC, sleep-current ladder, doc and fab refresh
Design (Rev 1.0, content current to 2026-09-21):
- DW01A: R83 100R supply filter with C7 on the pin side, C34 2.2n on CS
- F2 0805L075WR PPTC in series with J6 pin 12; CR3 now on the fused net
- U14 RV-8263-C7 alternate RTC footprint (DNP) with a project symbol library
- USB_STAT ladder rescaled x10 (R70 1M, R17 2M, R67 510k, R71 200k, C23 0.1u)
  and R57 10M: about 15 uA less sleep current
- R15 1M, C2 25 V part, 22 uF to Basic C45783, R14 to Basic C22939
- H6 mounting hole, H5 moved, single 5.30 x 1.10 mm neck slot, wider VBUS trunk
- Silkscreen: GitHub QR now points at silkscreen-pcb, battery warning at the
  cut line, display part number GDEQ0426T82-FT01C, LED current 13.3 mA
- Symbol fields corrected (AO3401A, IRLML6346, 1N5819HW, TVS, ESD arrays,
  connectors); local simulation-model paths removed

Fabrication:
- production/ regenerated with the Fabrication Toolkit and verified against
  the saved board; bom_JLC_upload_v4_optimized.csv renamed jlc_bom.csv,
  v3 removed; other-fab files regenerated
- part_fields.csv, BOM.md and the hand-build BOM updated

Docs:
- README rewritten as a JLCPCB ordering guide for beginners, with a real
  quote, glossary, configuration groups and the other-fab position
- HARDWARE.md: firmware contract, enclosure dimensions, new ladder levels,
  battery-protection and mounting notes; schematic screenshots, PDFs, board
  renders and a STEP model regenerated
- DESIGN_REVIEW.md status banner; simulations/ and the old de-link parts
  sheet removed
Parts:
- added C34: 2.2n, Capacitor_SMD:C_0603_1608Metric_Pad1.08x0.95mm_HandSolder, B.Cu at (90.6, 72.3)
- added F2: 0805L075WR, Fuse:Fuse_0805_2012Metric_Pad1.15x1.40mm_HandSolder, B.Cu at (87.0, 57.0)
- added H6: MountingHole_Pad, MountingHole:MountingHole_2.2mm_M2_DIN965_Pad_TopBottom, B.Cu at (69.2, 117.5)
- added R83: 100, Resistor_SMD:R_0603_1608Metric_Pad0.98x0.95mm_HandSolder, B.Cu at (88.4, 83.9)
- added U14: RV-8263-C7, Package_SON:MicroCrystal_C7_SON-8_1.5x3.2mm_P0.9mm, B.Cu at (63.9, 118.0)
- C18, C19: value 1u -> 1u/50V
- C2: value 10u -> 10u/25V
- C23: value 2.2n -> 0.1u
- C24, C31: value 100n -> 0.1u
- R15: value 10k -> 1M
- R17: value 150k -> 2M
- R57: value 1M -> 10M
- R67: value 56k -> 510k
- R70: value 100k -> 1M
- R71: value 22k -> 200k
- moved R56 2.20 mm to (90.8, 70.8), turned to 180 degrees
- moved R47 1.91 mm to (63.0, 114.6)
- moved R48 1.39 mm to (66.8, 114.4)
- moved H5 0.54 mm to (94.6, 72.2)
- moved R79 0.39 mm to (88.7, 87.1)
- moved Q1 0.15 mm to (86.5, 72.0)
Connections:
- C7 pad 1: P+ -> Net-(U5-VCC)
- CR3 pad 1: P+ -> /P+_FUSE
- J6 pad 12: P+ -> /P+_FUSE
- U5 pad 5: P+ -> Net-(U5-VCC)
Routing:
- net /P+_FUSE: track 0.00 -> 28.7 mm, vias 0 -> 2
- net P+: track 85.0 -> 59.2 mm, vias 6 -> 5
- net Net-(U5-CS): track 3.88 -> 17.4 mm, vias 0 -> 2
- net Net-(U5-VCC): track 0.00 -> 8.45 mm
- net I2C_SCL: track 178.6 -> 185.6 mm, vias 5 -> 6
- net 3V3: track 379.1 -> 385.4 mm
- net B-: track 35.4 -> 39.4 mm
- net UNUSED_GPIO_46: track 92.6 -> 95.2 mm
- net Net-(Q3-G): track 6.43 -> 8.81 mm
- net I2C_SDA: track 184.0 -> 181.9 mm
- net Net-(Q3-D): track 7.27 -> 8.40 mm
- net GND: track 48.8 -> 49.7 mm, vias 68 -> 69
- net UNUSED_GPIO_3: track 69.6 -> 68.7 mm
- net USB_VBUS: track 69.8 -> 70.6 mm
- net C-: track 187.9 -> 188.5 mm
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Other:
- outline, holes or cut-outs redrawn
- board text added: "GDEQ0426T82-FT01C: 1 - C+ 2 - C- 3 - NC 4 - NC 5 - W+ 6 - W-"
- board text added: "GDEQ0426T82-FT01C: 1 - GND 2 - VDD 3 - RST 4 - INT 5 - SDA 6 - SCL"
- board text added: "made with love by Ian C by several, including:"
- board text added: "supported"
- board text removed: "GDEQ426T82FT01: 1 - C+ 2 - C- 3 - NC 4 - NC 5 - W+ 6 - W-"
- board text removed: "GDEQ426T82FT01: 1 - GND 2 - VDD 3 - RST 4 - INT 5 - SDA 6 - SCL"
- board text removed: "made with love by Ian C supported by several, including:"
- board text removed: "this long end of the board can be cut for smaller displays if so, unpopulate R36 and R73 and then, populate R72/R74 this will swap power button to UP2 depopulate SW5 (DOWN2) if you please"
